File: Tomie2-Macro-Pad/Tomie2-Macro-Pad.kicad_pcb (KiCad board)
At the start: 2 copper layers, 76.2 x 38.1 mm, 24 parts, among them SW1 SW_Push, U1 ATmega32U4-A, Y1 16MHz

Commit message: PCB Finished
Parts:
- added G***: LOGO, LOGO, F.Cu at (56.4, 122.2)
- moved C2 2.11 mm to (65.6, 95.7)
- moved C1 2.11 mm to (74.6, 95.6)
- moved Y1 2.11 mm to (70.1, 95.7)
- moved C4 1.24 mm to (61.3, 101.0)
- moved R1 1.24 mm to (58.3, 101.0)
- moved C3 1.20 mm to (58.6, 108.2)
Connections:
- U1 pad 27: unconnected-(U1-Pad27) -> ROW0
- U1 pad 28: unconnected-(U1-Pad28) -> COL1
- U1 pad 29: unconnected-(U1-Pad29) -> COL0
- U1 pad 30: unconnected-(U1-Pad30) -> ROW1
Routing:
- net GND: track 59.4 -> 144.8 mm
- net +5V: track 15.4 -> 95.4 mm, vias 0 -> 5
- net COL1: track 0.00 -> 51.4 mm
- net ROW1: track 0.00 -> 47.3 mm
- net COL0: track 0.00 -> 32.0 mm
- net ROW0: track 19.6 -> 46.4 mm
- net Net-(R1-Pad2): track 21.8 -> 39.2 mm
- net Net-(C2-Pad2): track 3.42 -> 14.2 mm
- net Net-(C3-Pad1): track 0.00 -> 4.96 mm
- net Net-(R4-Pad1): track 0.00 -> 4.29 mm
- net Net-(C1-Pad2): track 9.83 -> 12.5 mm
- added copper zone on B.Cu, net GND
